File: rosco_m68k_keyboard-2.kicad_sch (KiCad schematic)
At the start: 166 parts, among them J1 Conn_01x04_Pin, J2 Conn_02x03_Odd_Even, J3 Conn_02x08_Odd_Even, J5 Conn_02x02_Odd_Even, K0 ESC, K1 !,1, K10 ),0, K11 _,-, K12 +,=, K13 BACKSPACE ⌫, K14 F1, K15 TAB ⇥, K16 Q, K17 W, K18 E, K19 R, K2 @,2, K20 T, K21 Y, K22 U, K23 I, K24 O, K25 P, K26 {,[, K27 },], K28 ⏎, K29 F2, K3 £,3, K30 CAPSLOCK, K31 A, K32 S, K33 D, K34 F, K35 G, K36 H, K37 J, K38 K, K39 L, K4 $,4, K40 :,;, K41 ",', K42 |,\, K43 F3, K44 SHIFT ⇧, K45 ~~,`, K46 Z, K47 X, K48 C, K49 V, K5 %,5, K50 B, K51 N, K52 M, K53 <,,, K54 >,., K55 ?,/, K56 SHIFT ⇧, K57 F4, K58 CTRL ^, K59 ⌘, K6 ^,6, K60 r, K61 Blank, K62 r, K63 ⌘, K64 ⌥, K65 CTRL ^, K66 F5, K7 &,7, K8 *,8, K9 (,9, SW1 Reset_SW, U1 ATmega64A-A, Y1 Crystal

Commit message: working
Parts:
- D67, D68, D69, D70, H1, H2, H3, H4, J1, J2, J3, J5, K0, K1, K10, K11, K12, K13, K14, K15, K16, K17, K18, K19, K2, K20, K21, K22, K23, K24, K25, K26, K27, K28, K29, K3, K30, K31, K32, K33, K34, K35, K36, K37, K38, K39, K4, K40, K41, K42, K43, K44, K45, K46, K47, K48, K49, K5, K50, K51, K52, K53, K54, K55, K56, K57, K58, K59, K6, K60, K61, K62, K63, K64, K65, K66, K7, K8, K9: now left out of the parts list
Connections:
- net A1: now also J3.13 (Pin_13), U1.31 (PD6); no longer J3.4 (Pin_4), U1.60 (PF1)
- net A2: now also J3.15 (Pin_15), U1.32 (PD7); no longer J3.2 (Pin_2), U1.61 (PF0)
- net AVEC: now also J3.3 (Pin_3), U1.26 (PD1); no longer J3.14 (Pin_14), U1.55 (PF6)
- net D0: now also J3.2 (Pin_2), U1.61 (PF0); no longer J3.1 (Pin_1), U1.25 (PD0)
- net D1: now also J3.4 (Pin_4), U1.60 (PF1); no longer J3.3 (Pin_3), U1.26 (PD1)
- net D2: now also J3.6 (Pin_6), U1.59 (PF2); no longer J3.5 (Pin_5), U1.27 (PD2)
- net D3: now also J3.8 (Pin_8), U1.58 (PF3); no longer J3.7 (Pin_7), U1.28 (PD3)
- net D4: now also J3.10 (Pin_10), U1.57 (PF4); no longer J3.9 (Pin_9), U1.29 (PD4)
- net D5: now also J3.12 (Pin_12), U1.56 (PF5); no longer J3.11 (Pin_11), U1.30 (PD5)
- net D6: now also J3.14 (Pin_14), U1.55 (PF6); no longer J3.13 (Pin_13), U1.31 (PD6)
- net D7: now also J3.16 (Pin_16), U1.54 (PF7); no longer J3.15 (Pin_15), U1.32 (PD7)
- net DTACK: now also J3.7 (Pin_7), U1.28 (PD3); no longer J3.10 (Pin_10), U1.57 (PF4)
- net IACK: now also J3.5 (Pin_5), U1.27 (PD2); no longer J3.12 (Pin_12), U1.56 (PF5)
- net IRQ: now also J3.9 (Pin_9), U1.29 (PD4); no longer J3.8 (Pin_8), U1.58 (PF3)
- net RW: now also J3.11 (Pin_11), U1.30 (PD5); no longer J3.6 (Pin_6), U1.59 (PF2)
- net SELECT: now also J3.1 (Pin_1), U1.25 (PD0); no longer J3.16 (Pin_16), U1.54 (PF7)

Commit message: Tidy up PCB
Parts:
- added J3: Conn_02x08_Odd_Even, Connector_PinHeader_2.54mm:PinHeader_2x08_P2.54mm_Vertical, symbol Connector_Generic:Conn_02x08_Odd_Even
- renumbered J3 to J4
Connections:
- net GND: now also J4.11 (Pin_11), J4.12 (Pin_12), J4.3 (Pin_3), J4.5 (Pin_5), J4.7 (Pin_7), J4.9 (Pin_9), J3.1 (Pin_1), J3.10 (Pin_10), J3.11 (Pin_11), J3.13 (Pin_13), J3.15 (Pin_15), J3.8 (Pin_8)
- net VCC: now also J4.1 (Pin_1), J3.2 (Pin_2), J3.5 (Pin_5)
- net A1 renamed AUX_D5
- net AUX_D5: now also U1.30 (PD5); no longer U1.31 (PD6)
- net A2 renamed AUX_D4
- net AUX_D4: now also U1.29 (PD4); no longer U1.32 (PD7)
- net AUX0: no longer names the net of U1.33 (PG0)
- net AUX1: no longer names the net of U1.34 (PG1)
- net AUX2: no longer names the net of U1.43 (PG2)
- net AUX3: no longer names the net of U1.18 (PG3)
- net AUX4: no longer names the net of U1.19 (PG4)
- net AVEC renamed SDA
- net SDA: now also J3.6 (Pin_6); no longer J4.3 (Pin_3)
- net D0 renamed AUX_F0
- net D1 renamed AUX_F1
- net D2 renamed AUX_F2
- net D3 renamed AUX_F3
- net D4 renamed AUX_F4
- net D5 renamed X_JP_I
- net X_JP_I: now also J3.12 (Pin_12); no longer J4.12 (Pin_12)
- net D6 renamed AUX_D6
- net AUX_D6: now also U1.31 (PD6); no longer U1.55 (PF6)
- net D7 renamed AUX_D7
- net AUX_D7: now also U1.32 (PD7); no longer U1.54 (PF7)
- net DTACK renamed TXD
- net TXD: now also J3.7 (Pin_7); no longer J4.7 (Pin_7)
- net IACK renamed RXD
- net RXD: now also J3.9 (Pin_9); no longer J4.5 (Pin_5)
- removed net IRQ: J4.9 (Pin_9), U1.29 (PD4)
- removed net RW: J4.11 (Pin_11), U1.30 (PD5)
- net SELECT renamed SCL
- net SCL: now also J3.4 (Pin_4); no longer J4.1 (Pin_1)
- new net UART_MODE_JP_I: J3.14 (Pin_14), U1.54 (PF7)
- new net UART_SPEED_JP_I: J3.16 (Pin_16), U1.55 (PF6)
- no-connect marks 2 -> 8
Other:
- note added: "AUX - NOT NORMALLY POPULATED"
- note added: "AUX_POWER"
- note added: "EXT_CTRL (SPI)"
- note added: "INTERFACE"
- note added: "ISP"
- note added: "NOT NORMALLY POPULATED"
- moved on the sheet: C6, C7, D60, D67, D68, D69, D70, J1, J2, J4, J5, K60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
